File: cpu.sch (KiCad schematic (older format))
At the start: 24 parts, among them SW1 RESET, SW2 STEP, U1 Z80CPU, U2 74HC04, Y1 7.3728MHz

Commit message: Change to 7 mils clearance to make cheaper
7 mils seems to be the minimum clearance for the cheap board houses. So
reworked the board to match.
Parts:
- SW1, SW2: footprint Buttons_Switches_SMD:SW_SPST_B3SL-1002P -> Buttons_Switches_ThroughHole:SW_PUSH_SMALL
Changed lines of the file:
@@
 	7550 1850 7450 1850
 Wire Wire Line
-	7450 1400 7450 1850
+	7450 1850 7450 1400
 Text Label 4150 1400 0    60   ~ 0
 ~RESET
@@
 F 0 "SW1" H 3700 1510 50  0000 C CNN
 F 1 "RESET" H 3550 1320 50  0000 C CNN
-F 2 "Buttons_Switches_SMD:SW_SPST_B3SL-1002P" H 3550 1400 50  0001 C CNN
+F 2 "Buttons_Switches_ThroughHole:SW_PUSH_SMALL" H 3550 1400 50  0001 C CNN
 F 3 "" H 3550 1400 50  0000 C CNN
 	1    3550 1400
@@
 $EndComp
 Wire Wire Line
-	3850 1400 7450 1400
+	7450 1400 3850 1400
 $Comp
 L 74HC04 U2
@@
 F 0 "SW2" H 3200 7160 50  0000 C CNN
 F 1 "STEP" H 3050 6970 50  0000 C CNN
-F 2 "Buttons_Switches_SMD:SW_SPST_B3SL-1002P" H 3050 7050 50  0001 C CNN
+F 2 "Buttons_Switches_ThroughHole:SW_PUSH_SMALL" H 3050 7050 50  0001 C CNN
 F 3 "" H 3050 7050 50  0000 C CNN
 	1    3050 7050
